Commit message: Final thesis code

File: urdfs/robot.urdf (robot description, URDF)
Before this commit: robot myrobot, 11 links, 10 joints
Joints:
- joint camera_joint: origin xyz=0.05 0 0.02 rpy=0 0 0 -> xyz=0.025 0 0.02 rpy=0 0 0

File: urdfs/robot.urdf.xacro (robot description, xacro)
@@ -51,5 +51,5 @@
   <joint name="camera_joint" type="fixed">
     <axis xyz="0 1 0" />
-    <origin xyz="${pan_tilt_diam} 0 0.02" rpy="0 0 0"/>
+    <origin xyz="${pan_tilt_diam/2} 0 0.02" rpy="0 0 0"/>
     <parent link="pan_tilt_link"/>
     <child link="camera_link"/>
